Commit message: small changes

File: VirtualRobot/data/robots/aurmr/tahoma_copy.urdf (robot description, URDF)
Before this commit: robot tahoma, 38 links, 37 joints
Links:
- removed link arm_base
- removed link arm_base_link
- removed link arm_base_link_inertia
- removed link arm_flange
- removed link arm_forearm_link
- removed link arm_shoulder_link
- removed link arm_tool0
- removed link arm_upper_arm_link
- removed link arm_wrist_1_link
- removed link arm_wrist_2_link
- removed link arm_wrist_3_link
- removed link back_left_caster
- removed link back_right_caster
- removed link base_link
- removed link camera_base
- removed link camera_beam_lower
- removed link camera_body
- removed link camera_lower_left_mount
- removed link camera_lower_right_mount
- removed link camera_upper_mount
- removed link camera_visor
- removed link cantilever
- removed link control_box
- removed link control_box_mount
- removed link coupling
- removed link epick_end_effector
- removed link front_left_caster
- removed link front_right_caster
- removed link gripper_base_link
- removed link left_light_panel
- removed link left_light_panel_emitter
- removed link right_light_panel
- removed link right_light_panel_emitter
- removed link robot_plate
- removed link stand
- removed link stand_brace
- removed link stand_upright
Joints:
- removed joint $hand__end_effector_joint
- removed joint arm_base_link-base_fixed_joint
- removed joint arm_base_link-base_link_inertia
- removed joint arm_elbow_joint
- removed joint arm_flange-tool0
- removed joint arm_shoulder_lift_joint
- removed joint arm_shoulder_pan_joint
- removed joint arm_tool0-coupling_joint
- removed joint arm_wrist_1_joint
- removed joint arm_wrist_2_joint
- removed joint arm_wrist_3-flange
- removed joint arm_wrist_3_joint
- removed joint base_joint
- removed joint camera_base_to_body
- removed joint camera_base_to_visor
- removed joint camera_beam_lower_camera_lower_left_mount_joint
- removed joint camera_beam_lower_camera_lower_right_mount_joint
- removed joint cantilever_camera_upper_mount_joint
- removed joint cantilever_robot_plate_joint
- removed joint control_box_mount_control_box_joint
- removed joint coupling_link_gripper_robotiq_arg2f_base_link_joint
- removed joint kinect_base_joint
- removed joint left_light_panel_left_light_panel_emitter_joint
- removed joint right_light_panel_right_light_panel_emitter_joint
- removed joint robot_plate_arm_base_link_joint
- removed joint stand_back_left_caster_joint
- removed joint stand_back_right_caster_joint
- removed joint stand_cantilever_joint
- removed joint stand_front_left_caster_joint
- removed joint stand_front_right_caster_joint
- removed joint stand_left_light_panel_joint
- removed joint stand_left_right_panel_joint
- removed joint stand_stand_upright_joint
- removed joint stand_upright_camera_beam_lower_joint
- removed joint stand_upright_robot_control_box_mount_joint
- removed joint stand_upright_stand_brace_joint

File: VirtualRobot/data/robots/aurmr/tahoma_test.urdf (robot description, URDF)
Before this commit: robot tahoma, 38 links, 37 joints
Links:
- link epick_end_effector: geometry collision cylinder length=0.017 radius=0.0225; visual cylinder length=0.017 radius=0.0225
Joints:
- joint coupling_link_gripper_robotiq_arg2f_base_link_joint: origin xyz=0 0 -0.034 rpy=0 0 0 -> xyz=0 0 0.017 rpy=0 0 0

Commit message: visu in front of bin E to H

File: VirtualRobot/data/robots/aurmr/tahoma_copy.urdf (robot description, URDF)
Before this commit: robot tahoma, 1 links, 1 joints
Links:
- added link arm_base
- added link arm_base_link
- added link arm_base_link_inertia, mass 4.0; collision mesh filename=package://ur_description/meshes/ur10e/collision/base.stl; visual mesh filename=package://ur_description/meshes/ur10e/visual/base_std.dae
- added link arm_flange
- added link arm_forearm_link, mass 4.321; collision mesh filename=package://ur_description/meshes/ur16e/collision/forearm.stl; visual mesh filename=package://ur_description/meshes/ur16e/visual/forearm_std.dae
- added link arm_shoulder_link, mass 7.369; collision mesh filename=package://ur_description/meshes/ur10e/collision/shoulder.stl; visual mesh filename=package://ur_description/meshes/ur10e/visual/shoulder_std.d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
- added link arm_tool0
- added link arm_upper_arm_link, mass 10.45; collision mesh filename=package://ur_description/meshes/ur16e/collision/upperarm.stl; visual mesh filename=package://ur_description/meshes/ur16e/visual/upperarm_std.d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
- added link arm_wrist_1_link, mass 2.18; collision mesh filename=package://ur_description/meshes/ur10e/collision/wrist1.stl; visual mesh filename=package://ur_description/meshes/ur10e/visual/wrist1_std.dae
- added link arm_wrist_2_link, mass 2.033; collision mesh filename=package://ur_description/meshes/ur10e/collision/wrist2.stl; visual mesh filename=package://ur_description/meshes/ur10e/visual/wrist2_std.dae
- added link arm_wrist_3_link, mass 0.907; collision mesh filename=package://ur_description/meshes/ur10e/collision/wrist3.stl; visual mesh filename=package://ur_description/meshes/ur10e/visual/wrist3_std.dae
- added link back_left_caster, mass 1.0; collision box size=0.09 0.1040 0.1225; visual mesh filename=package://tahoma_description/meshes/stand/caster.stl
- added link back_right_caster, mass 1.0; collision box size=0.09 0.1040 0.1225; visual mesh filename=package://tahoma_description/meshes/stand/caster.stl
- added link base_link
- added link camera_base; visual box size=0.026 0.103 0.039
- added link camera_beam_lower, mass 5; collision box size=0.045 1.25 0.045; visual mesh filename=package://tahoma_description/meshes/stand/camera_beam.stl
- added link camera_body; visual box size=0.0994 0.0996 0.023
- added link camera_lower_left_mount; collision box size=.1 .15 .15
- added link camera_lower_right_mount; collision box size=.1 .15 .15
- added link camera_upper_mount
- added link camera_visor; visual box size=0.026 0.101 0.037
- added link cantilever, mass 8; collision box size=.7260 .225 .09; visual mesh filename=package://tahoma_description/meshes/stand/cantilever.stl
- added link control_box, mass 7; collision box size=.46 .25 .44; visual mesh filename=package://tahoma_description/meshes/stand/control_box.stl
- added link control_box_mount, mass 3; collision box size=.585 .0602 .1790; visual mesh filename=package://tahoma_description/meshes/stand/control_box_mount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
- added link coupling; collision box size=.015 0.033 .056; collision cylinder length=.0169 radius=.0375
- added link epick_end_effector, mass 0.0001; collision cylinder length=0.017 radius=0.0225; visual cylinder length=0.017 radius=0.0225
- added link front_left_caster, mass 1.0; collision box size=0.09 0.1040 0.1225; visual mesh filename=package://tahoma_description/meshes/stand/caster.stl
- added link front_right_caster, mass 1.0; collision box size=0.09 0.1040 0.1225; visual mesh filename=package://tahoma_description/meshes/stand/caster.stl
- added link gripper_base_link, mass 0.745; collision cylinder length=0.08 radius=0.006; collision cylinder length=0.114 radius=0.035
- added link left_light_panel, mass 1.0; collision box size=1.21 .602 .01; visual box size=1.21 .602 .01
- added link left_light_panel_emitter; collision box size=1.17 .562 .00251; visual box size=1.17 .562 .00251
- added link right_light_panel, mass 1.0; collision box size=1.21 .602 .01; visual box size=1.21 .602 .01
- added link right_light_panel_emitter; collision box size=1.17 .562 .00251; visual box size=1.17 .562 .00251
- added link robot_plate, mass .5; collision box size=.225 .225 .0225; visual mesh filename=package://tahoma_description/meshes/stand/robot_plate.stl
- added link stand, mass 10.0; collision box size=.09 1.53 .045; collision box size=.9 .09 .0562
- added link stand_brace, mass 5; collision box size=.102 1.4390 .4934; visual mesh filename=package://tahoma_description/meshes/stand/stand_brace.stl
- added link stand_upright, mass 34; collision box size=.2298 .0450 1.89; collision box size=.2298 .0450 1.89
Joints:
- added joint $hand__end_effector_joint: type fixed, parent gripper_base_link, child epick_end_effector, origin xyz=0 0 0.187 rpy=0 0 0
- added joint arm_base_link-base_fixed_joint: type fixed, parent arm_base_link, child arm_base, origin xyz=0 0 0 rpy=0 0 3.141592653589793
- added joint arm_base_link-base_link_inertia: type fixed, parent arm_base_link, child arm_base_link_inertia, origin xyz=0 0 0 rpy=0 0 3.141592653589793
- added joint arm_elbow_joint: type revolute, parent arm_upper_arm_link, child arm_forearm_link, origin xyz=-0.478259666576996 0 0 rpy=3.140966205585682 3.14143866526404 3.141584703118312, axis 0 0 1, limit lower=-3.141592653589793 upper=3.141592653589793 effort=150.0 velocity=3.141592653589793
- added joint arm_flange-tool0: type fixed, parent arm_flange, child arm_tool0, origin xyz=0 0 0 rpy=1.5707963267948966 0 1.5707963267948966
- added joint arm_shoulder_lift_joint: type revolute, parent arm_shoulder_link, child arm_upper_arm_link, origin xyz=0.0001146488038115345 0 0 rpy=1.571149055019948 0 -2.842156630394906e-06, axis 0 0 1, limit lower=-6.283185307179586 upper=6.283185307179586 effort=330.0 velocity=2.0943951023931953
- added joint arm_shoulder_pan_joint: type revolute, parent arm_base_link_inertia, child arm_shoulder_link, origin xyz=0 0 0.1808582427003927 rpy=0 0 -5.226355219677126e-07, axis 0 0 1, limit lower=-6.283185307179586 upper=6.283185307179586 effort=330.0 velocity=2.0943951023931953
- added joint arm_tool0-coupling_joint: type fixed, parent arm_tool0, child coupling, origin xyz=0 0 -0.003 rpy=0 0 4.71238898038469
- added joint arm_wrist_1_joint: type revolute, parent arm_forearm_link, child arm_wrist_1_link, origin xyz=-0.3600303731229585 -0.001096754867652125 0.1741650928407709 rpy=0.006297130801998122 0.0009340032369312529 1.229979779393521e-06, axis 0 0 1, limit lower=-6.283185307179586 upper=6.283185307179586 effort=56.0 velocity=3.141592653589793
- added joint arm_wrist_2_joint: type revolute, parent arm_wrist_1_link, child arm_wrist_2_link, origin xyz=5.900314979285639e-05 -0.1197777051587798 0.0002253351762985995 rpy=1.568915050891635 0 1.761825868220462e-06, axis 0 0 1, limit lower=-6.283185307179586 upper=6.283185307179586 effort=56.0 velocity=3.141592653589793
- added joint arm_wrist_3-flange: type fixed, parent arm_wrist_3_link, child arm_flange, origin xyz=0 0 0 rpy=0 -1.5707963267948966 -1.5707963267948966
- added joint arm_wrist_3_joint: type revolute, parent arm_wrist_2_link, child arm_wrist_3_link, origin xyz=9.510304711030174e-05 0.115763931390055 -7.780349503190604e-05 rpy=1.570124239363319 3.141592653589793 -3.141592198139823, axis 0 0 1, limit lower=-6.283185307179586 upper=6.283185307179586 effort=56.0 velocity=3.141592653589793
- added joint base_joint: type fixed, parent base_link, child stand, origin xyz=0 0 0.15 rpy=0 0 0
- added joint camera_base_to_body: type fixed, parent camera_base, child camera_body, origin xyz=-0.0757 0. 0.008 rpy=0. 0. 0.
- added joint camera_base_to_visor: type fixed, parent camera_base, child camera_visor, origin xyz=0. 0. 0. rpy=0. 0. 0.
- added joint camera_beam_lower_camera_lower_left_mount_joint: type fixed, parent camera_beam_lower, child camera_lower_left_mount, origin xyz=0.02 0.2285 0.14 rpy=1.5707963267948966 0.2617993877991494 -0.1767088560700366
- added joint camera_beam_lower_camera_lower_right_mount_joint: type fixed, parent camera_beam_lower, child camera_lower_right_mount, origin xyz=0.02 -0.2285 0.14 rpy=1.5707963267948966 0.2617993877991494 0.1767088560700366
- added joint cantilever_camera_upper_mount_joint: type fixed, parent cantilever, child camera_upper_mount, origin xyz=.02 0 0.37 rpy=0 0.2617993877991494 0
- added joint cantilever_robot_plate_joint: type fixed, parent cantilever, child robot_plate, origin xyz=0.2505 0 -.015 rpy=0 0 0
- added joint control_box_mount_control_box_joint: type fixed, parent control_box_mount, child control_box, origin xyz=-.003 .1375 -0.13 rpy=0.05 0 3.141592653589793
- added joint coupling_link_gripper_robotiq_arg2f_base_link_joint: type fixed, parent coupling, child gripper_base_link, origin xyz=0 0 0.017 rpy=0 0 0
- added joint kinect_base_joint: type fixed, parent base_link, child camera_base, origin xyz=-0.245645 -0.011721185 1.41034 rpy=3.13764 3.12912 -3.12899
- added joint left_light_panel_left_light_panel_emitter_joint: type fixed, parent left_light_panel, child left_light_panel_emitter
- added joint right_light_panel_right_light_panel_emitter_joint: type fixed, parent right_light_panel, child right_light_panel_emitter
- added joint robot_plate_arm_base_link_joint: type fixed, parent robot_plate, child arm_base_link, origin xyz=0 0.00175 -0.00885 rpy=0 3.141592653589793 4.71238898038469
- added joint stand_back_left_caster_joint: type fixed, parent stand, child back_left_caster, origin xyz=-.405 .7025 -0.1 rpy=0 0 0
- added joint stand_back_right_caster_joint: type fixed, parent stand, child back_right_caster, origin xyz=-.405 -.7375 -0.1 rpy=0 0 0
- added joint stand_cantilever_joint: type fixed, parent stand_upright, child cantilever, origin xyz=.0775 0  0.9442 rpy=0 0 0
- added joint stand_front_left_caster_joint: type fixed, parent stand, child front_left_caster, origin xyz=.405 .7025 -0.1 rpy=0 0 0
- added joint stand_front_right_caster_joint: type fixed, parent stand, child front_right_caster, origin xyz=.405 -.7375 -0.1 rpy=0 0 0
- added joint stand_left_light_panel_joint: type fixed, parent stand_upright, child left_light_panel, origin xyz=-.2625 .35 .25 rpy=0 1.5707963267948966 0
- added joint stand_left_right_panel_joint: type fixed, parent stand_upright, child right_light_panel, origin xyz=-.2625 -.35 .25 rpy=0 1.5707963267948966 0
- added joint stand_stand_upright_joint: type fixed, parent stand, child stand_upright, origin xyz=-.12 0 .95 rpy=0 0 0
- added joint stand_upright_camera_beam_lower_joint: type fixed, parent stand_upright, child camera_beam_lower, origin xyz=-.1225 0 .193 rpy=0 0 0
- added joint stand_upright_robot_control_box_mount_joint: type fixed, parent stand_upright, child control_box_mount, origin xyz=-.1725 .7475 .21 rpy=0 0 0
- added joint stand_upright_stand_brace_joint: type fixed, parent stand_upright, child stand_brace, origin xyz=-.24 0 -.59 rpy=0 0 0

File: VirtualRobot/data/robots/aurmr/tahoma_test.urdf (robot description, URDF)
Before this commit: robot tahoma, 38 links, 37 joints
Links:
- link back_left_caster: geometry collision mesh filename=package://tahoma_description/meshes/stand/caster_col.stl; visual mesh filename=package://tahoma_description/meshes/stand/caster.stl
- link back_right_caster: geometry collision mesh filename=package://tahoma_description/meshes/stand/caster_col.stl; visual mesh filename=package://tahoma_description/meshes/stand/caster.stl
- link camera_base: geometry visual mesh filename=package://tahoma_description/meshes/stand/camera_base.stl
- link camera_beam_lower: geometry collision mesh filename=package://tahoma_description/meshes/stand/camera_beam_col.s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; visual mesh filename=package://tahoma_description/meshes/stand/camera_beam.stl
- link camera_body: geometry visual mesh filename=package://tahoma_description/meshes/stand/camera_body.stl
- link camera_lower_left_mount: geometry collision mesh filename=package://tahoma_description/meshes/stand/camera_lower_left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
- link camera_lower_right_mount: geometry collision mesh filename=package://tahoma_description/meshes/stand/camera_lower_righ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
- link camera_visor: geometry visual mesh filename=package://tahoma_description/meshes/stand/camera_visor.stl
- link cantilever: geometry collision mesh filename=package://tahoma_description/meshes/stand/cantilever_col.stl; visual mesh filename=package://tahoma_description/meshes/stand/cantilever.stl
- link control_box: geometry collision mesh filename=package://tahoma_description/meshes/stand/control_box_col.s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; visual mesh filename=package://tahoma_description/meshes/stand/control_box.stl
- link control_box_mount: geometry collision mesh filename=package://tahoma_description/meshes/stand/control_box_mount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; visual mesh filename=package://tahoma_description/meshes/stand/control_box_mount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
- link coupling: geometry collision mesh filename=package://robotiq_2f_85_gripper_visualization/meshes/visual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; visual mesh filename=package://robotiq_2f_85_gripper_visualization/meshes/visual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
- link epick_end_effector: geometry collision mesh filename=package://tahoma_description/meshes/stand/epick_end_effecto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; visual mesh filename=package://tahoma_description/meshes/stand/epick_end_effecto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
- link front_left_caster: geometry collision mesh filename=package://tahoma_description/meshes/stand/caster_col.stl; visual mesh filename=package://tahoma_description/meshes/stand/caster.stl
- link front_right_caster: geometry collision mesh filename=package://tahoma_description/meshes/stand/caster_col.stl; visual mesh filename=package://tahoma_description/meshes/stand/caster.stl
- link gripper_base_link: geometry collision mesh filename=package://robotiq_epick_visualization/meshes/visual/gripper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; visual mesh filename=package://robotiq_epick_visualization/meshes/visual/gripper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 scale=0.001 0.001 0.001
- link left_light_panel: geometry collision mesh filename=package://tahoma_description/meshes/stand/light_panel.stl; visual mesh filename=package://tahoma_description/meshes/stand/light_panel.stl
- link left_light_panel_emitter: geometry collision mesh filename=package://tahoma_description/meshes/stand/light_panel_emitt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; visual mesh filename=package://tahoma_description/meshes/stand/light_panel_emitt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
- link right_light_panel: geometry collision mesh filename=package://tahoma_description/meshes/stand/light_panel.stl; visual mesh filename=package://tahoma_description/meshes/stand/light_panel.stl
- link right_light_panel_emitter: geometry collision mesh filename=package://tahoma_description/meshes/stand/light_panel_emitt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; visual mesh filename=package://tahoma_description/meshes/stand/light_panel_emitt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
- link robot_plate: geometry collision mesh filename=package://tahoma_description/meshes/stand/robot_plate_col.s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; visual mesh filename=package://tahoma_description/meshes/stand/robot_plate.stl
- link stand: geometry collision mesh filename=package://tahoma_description/meshes/stand/stand_col.stl; visual mesh filename=package://tahoma_description/meshes/stand/stand_base.stl
- link stand_brace: geometry collision mesh filename=package://tahoma_description/meshes/stand/stand_brace_col.s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; visual mesh filename=package://tahoma_description/meshes/stand/stand_brace.stl
- link stand_upright: geometry collision mesh filename=package://tahoma_description/meshes/stand/stand_upright_col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; visual mesh filename=package://tahoma_description/meshes/stand/stand_upright.stl
